File: eco_devkit/mcu.kicad_sch (KiCad schematic)
At the start: 0 parts

Commit message: Update mcu.kicad_sch
Parts:
- added U1: RP2350B-QFN80, symbol rp2350b-qfn80:RP2350B-QFN80
Connections:
- new net GND: U1.4 (GND), U1.81 (GND)
- new net VCC: U1.5 (VCC)

Commit message: Update mcu.kicad_sch
Parts:
- removed U1: RP2350B-QFN80, symbol rp2350b-qfn80:RP2350B-QFN80
- added C1, C19, C5: 10u, symbol Device:C
- added C10, C6, C7, C9: 4.7u, symbol Device:C
- added C11, C12, C13, C14, C15, C16, C17, C18, C2, C20, C21, C8: 100n, symbol Device:C
- added C3, C4: 15p, symbol Device:C
- added FLASH_MEMORY_8MB: ~, Package_SON:WSON-8-1EP_6x5mm_P1.27mm_EP3.4x4.3mm, symbol rp2350b-qfn80:Flash_Memory_8MB
- added H1, H2, H3, H4: MountingHole, symbol Mechanical:MountingHole
- added J1, J2: Conn_02x26_Odd_Even, Connector_PinHeader_2.54mm:PinHeader_2x26_P2.54mm_Vertical, symbol Connector_Generic:Conn_02x26_Odd_Even
- added L1: 3.3u, symbol Device:L
- added NCP117: ~, symbol rp2350b-qfn80:NCP1117
- added P1: USB_C_Plug_USB2.0, symbol Connector:USB_C_Plug_USB2.0
- added R1, R9: DNF, symbol Device:R
- added R10: 0, symbol Device:R
- added R2, R4, R6: 1k, symbol Device:R
- added R3: R3, symbol Device:R
- added R7, R8: 27, symbol Device:R
- added RP2350B: ~, symbol rp2350b-qfn80:RP2350B-QFN80
- added SW1, SW2: SW_Push, symbol Switch:SW_Push
- added Y1: Crystal_GND24, symbol Device:Crystal_GND24
Connections:
- net GND: now also C1.2, C10.2, C11.2, C12.2, C13.2, C14.2, C15.2, C16.2, C17.2, C18.2, C19.2, C2.2, C20.2, C21.2, C3.1, C4.1, C5.2, C6.2, C7.2, C8.2, C9.2, FLASH_MEMORY_8MB.4 (GND), J1.1 (Pin_1), J1.11 (Pin_11), J1.13 (Pin_13), J1.15 (Pin_15), J1.17 (Pin_17), J1.19 (Pin_19), J1.21 (Pin_21), J1.23 (Pin_23), J1.25 (Pin_25), J1.27 (Pin_27), J1.29 (Pin_29), J1.3 (Pin_3), J1.31 (Pin_31), J1.33 (Pin_33), J1.35 (Pin_35), J1.37 (Pin_37), J1.39 (Pin_39), J1.41 (Pin_41), J1.43 (Pin_43), J1.45 (Pin_45), J1.47 (Pin_47), J1.49 (Pin_49), J1.5 (Pin_5), J1.51 (Pin_51), J1.7 (Pin_7), J1.9 (Pin_9), J2.10 (Pin_10), J2.12 (Pin_12), J2.14 (Pin_14), J2.16 (Pin_16), J2.18 (Pin_18), J2.2 (Pin_2), J2.20 (Pin_20), J2.22 (Pin_22), J2.24 (Pin_24), J2.26 (Pin_26), J2.28 (Pin_28), J2.30 (Pin_30), J2.32 (Pin_32), J2.34 (Pin_34), J2.36 (Pin_36), J2.38 (Pin_38), J2.4 (Pin_4), J2.40 (Pin_40), J2.42 (Pin_42), J2.44 (Pin_44), J2.46 (Pin_46), J2.48 (Pin_48), J2.50 (Pin_50), J2.52 (Pin_52), J2.6 (Pin_6), J2.8 (Pin_8), NCP117.1 (GND), P1.A1 (GND), P1.A12 (GND), P1.B1 (GND), P1.B12 (GND), P1.S1 (SHIELD), R4.1, RP2350B.62 (VREG_PGND), RP2350B.81 (GND), SW1.1, Y1.2, Y1.4
- new net: C9.1, R3.2, RP2350B.61 (VREG_AVDD)
- new net: R8.1, RP2350B.66 (USB_DM)
- new net: R7.1, RP2350B.67 (USB_DP)
- new net: R6.2, RP2350B.75 (QSPI_SS)
- new net: C4.2, R2.1, Y1.3
- new net: R4.2, SW2.1
- new net +1V1: C7.1, L1.1, RP2350B.65 (VREG_FB)
- new net +1v1: C10.1, C11.1, C8.1, RP2350B.10 (DVDD), RP2350B.32 (DVDD), RP2350B.51 (DVDD)
- new net +3.3V: C6.1, R3.1, RP2350B.64 (VREG_VIN)
- new net +3V3: C19.1, C2.1, C5.1, FLASH_MEMORY_8MB.8 (VCC), J1.2 (Pin_2), NCP117.2 (VO), R1.1
- new net +3v3: C12.1, C13.1, C14.1, C15.1, C16.1, C17.1, C18.1, C20.1, C21.1, RP2350B.15 (IOVDD), RP2350B.24 (IOVDD), RP2350B.29 (IOVDD), RP2350B.41 (IOVDD), RP2350B.5 (IOVDD), RP2350B.50 (IOVDD), RP2350B.59 (ADC_AVDD), RP2350B.60 (IOVDD), RP2350B.68 (USB_OTP_VDD), RP2350B.69 (QSPI_IOVDD), RP2350B.76 (IOVDD)
- new net FLASH_SS: FLASH_MEMORY_8MB.1 (/CS), R1.2, R10.2, R9.2
- new net GPIO0: J1.4 (Pin_4), R9.1, RP2350B.77 (GPIO0)
- new net GPIO1: J1.6 (Pin_6), RP2350B.78 (GPIO1)
- new net GPIO10: J1.24 (Pin_24), RP2350B.8 (GPIO10)
- new net GPIO11: J1.26 (Pin_26), RP2350B.9 (GPIO11)
- new net GPIO12: J1.28 (Pin_28), RP2350B.11 (GPIO12)
- new net GPIO13: J1.30 (Pin_30), RP2350B.12 (GPIO13)
- new net GPIO14: J1.32 (Pin_32), RP2350B.13 (GPIO14)
- new net GPIO15: J1.34 (Pin_34), RP2350B.14 (GPIO15)
- new net GPIO16: J1.36 (Pin_36), RP2350B.16 (GPIO16)
- new net GPIO17: J1.38 (Pin_38), RP2350B.17 (GPIO17)
- new net GPIO18: J1.40 (Pin_40), RP2350B.18 (GPIO18)
- new net GPIO19: J1.42 (Pin_42), RP2350B.19 (GPIO19)
- new net GPIO2: J1.8 (Pin_8)
- new net GPIO20: J1.44 (Pin_44), RP2350B.20 (GPIO20)
- new net GPIO21: J1.46 (Pin_46), RP2350B.21 (GPIO21)
- new net GPIO22: J1.48 (Pin_48), RP2350B.22 (GPIO22)
- new net GPIO23: J1.50 (Pin_50), RP2350B.23 (GPIO23)
- new net GPIO24: J1.52 (Pin_52), RP2350B.25 (GPIO24)
- new net GPIO25: J2.51 (Pin_51), RP2350B.26 (GPIO25)
- new net GPIO26: J2.49 (Pin_49), RP2350B.27 (GPIO26)
- new net GPIO27: J2.47 (Pin_47), RP2350B.28 (GPIO27)
- new net GPIO28: J2.39 (Pin_39), RP2350B.36 (GPIO28)
- new net GPIO29: J2.37 (Pin_37), RP2350B.37 (GPIO29)
- new net GPIO3: J1.10 (Pin_10), RP2350B.80 (GPIO3)
- new net GPIO30: J2.35 (Pin_35), RP2350B.38 (GPIO30)
- new net GPIO31: J2.33 (Pin_33), RP2350B.39 (GPIO31)
- new net GPIO32: J2.31 (Pin_31), RP2350B.40 (GPIO32)
- new net GPIO33: J2.29 (Pin_29), RP2350B.42 (GPIO33)
- new net GPIO34: J2.27 (Pin_27), RP2350B.43 (GPIO34)
- new net GPIO35: J2.25 (Pin_25), RP2350B.44 (GPIO35)
- new net GPIO36: J2.23 (Pin_23), RP2350B.45 (GPIO36)
- new net GPIO37: J2.21 (Pin_21), RP2350B.46 (GPIO37)
- new net GPIO38: J2.19 (Pin_19), RP2350B.47 (GPIO38)
- new net GPIO39: J2.17 (Pin_17), RP2350B.48 (GPIO39)
- new net GPIO4: J1.12 (Pin_12), RP2350B.1 (GPIO4), RP2350B.79 (GPIO2)
- new net GPIO40_ADC0: J2.15 (Pin_15), RP2350B.49 (GPIO40_ADC0)
- new net GPIO41_ADC1: J2.13 (Pin_13), RP2350B.52 (GPIO41_ADC1)
- new net GPIO42_ADC2: J2.11 (Pin_11), RP2350B.53 (GPIO42_ADC2)
- new net GPIO43_ADC3: J2.9 (Pin_9), RP2350B.54 (GPIO43_ADC3)
- new net GPIO44_ADC4: J2.7 (Pin_7), RP2350B.55 (GPIO44_ADC4)
- new net GPIO45_ADC5: J2.5 (Pin_5), RP2350B.56 (GPIO45_ADC5)
- new net GPIO46_ADC6: J2.3 (Pin_3), RP2350B.57 (GPIO46_ADC6)
- new net GPIO47_ADC7: J2.1 (Pin_1), RP2350B.58 (GPIO47_ADC7)
- new net GPIO5: J1.14 (Pin_14), RP2350B.2 (GPIO5)
- new net GPIO6: J1.16 (Pin_16), RP2350B.3 (GPIO6)
- new net GPIO7: J1.18 (Pin_18), RP2350B.4 (GPIO7)
- new net GPIO8: J1.20 (Pin_20), RP2350B.6 (GPIO8)
- new net GPIO9: J1.22 (Pin_22), RP2350B.7 (GPIO9)
- new net QSPI_SCLK: FLASH_MEMORY_8MB.6 (CLK), RP2350B.71 (QSPI_SCLK)
- new net QSPI_SD0: FLASH_MEMORY_8MB.5 (DI_(IO0)), RP2350B.72 (QSPI_SD0)
- new net QSPI_SD1: FLASH_MEMORY_8MB.2 (DO_(IO1)), RP2350B.74 (QSPI_SD1)
- new net QSPI_SD2: FLASH_MEMORY_8MB.3 (/WP_(IO2)), RP2350B.73 (QSPI_SD2)
- new net QSPI_SD3: FLASH_MEMORY_8MB.7 (/HOLD_(IO3)), RP2350B.70 (QSPI_SD3)
- new net QSPI_SS: R10.1
- new net RUN: J2.41 (Pin_41), RP2350B.35 (RUN), SW2.2
- new net SWCLK: J2.45 (Pin_45), RP2350B.33 (SWCLK)
- new net SWD: J2.43 (Pin_43), RP2350B.34 (SWDIO)
- new net USB_BOOT: R6.1, SW1.2
- new net USB_D+: P1.A6 (D+), R7.2
- new net USB_D-: P1.A7 (D-), R8.2
- new net VBUS: C1.1, NCP117.3 (VI), P1.A4 (VBUS), P1.A9 (VBUS), P1.B4 (VBUS), P1.B9 (VBUS)
- new net VREG_LX: L1.2, RP2350B.63 (VREG_LX)
- new net XIN: C3.2, RP2350B.30 (XIN), Y1.1
- new net XOUT: R2.2, RP2350B.31 (XOUT)
- no-connect marks 0 -> 1
Other:
- note added: "1.2MHz Crystal"
- note added: "FLASH MEMORY 8MB"
- note added: "IOs"
- note added: "POWER USB-C"
- note added: "RP2350B"

Commit message: Update mcu.kicad_sch
Parts:
- removed C19: 10u, symbol Device:C
- removed J1, J2: Conn_02x26_Odd_Even, Connector_PinHeader_2.54mm:PinHeader_2x26_P2.54mm_Vertical, symbol Connector_Generic:Conn_02x26_Odd_Even
- removed P1: USB_C_Plug_USB2.0, symbol Connector:USB_C_Plug_USB2.0
- added D1: SB120, Diode_THT:D_DO-41_SOD81_P10.16mm_Horizontal, symbol Diode:SB120
- added J2, J3: Conn_01x26_Pin, Connector_PinHeader_2.54mm:PinHeader_1x26_P2.54mm_Vertical, symbol Connector:Conn_01x26_Pin
- added J4: USB_C_Receptacle_USB2.0_16P, symbol Connector:USB_C_Receptacle_USB2.0_16P
- added R1, R2: 5.1k, symbol Device:R_Small_US
- C1, C11, C12, C13, C14, C15, C16, C17, C18, C2, C6, C7, C8: footprint (none) -> Capacitor_SMD:C_0402_1005Metric
- C10: renamed from C9; footprint (none) -> Capacitor_SMD:C_0402_1005Metric
- C19: renamed from C20; footprint (none) -> Capacitor_SMD:C_0402_1005Metric
- C20: renamed from C21; footprint (none) -> Capacitor_SMD:C_0402_1005Metric
- C3: renamed from C5; footprint (none) -> Capacitor_SMD:C_0402_1005Metric
- C4: renamed from C3; footprint (none) -> Capacitor_SMD:C_0402_1005Metric
- C5: renamed from C4; footprint (none) -> Capacitor_SMD:C_0402_1005Metric
- C9: renamed from C10; footprint (none) -> Capacitor_SMD:C_0402_1005Metric
- R10: renamed from R7; footprint (none) -> Resistor_SMD:R_0402_1005Metric
- R11: renamed from R8; footprint (none) -> Resistor_SMD:R_0402_1005Metric
- R3: renamed from R9; footprint (none) -> Resistor_SMD:R_0402_1005Metric
- R4: renamed from R10; footprint (none) -> Resistor_SMD:R_0402_1005Metric
- R5: renamed from R1; footprint (none) -> Resistor_SMD:R_0402_1005Metric
- R6: renamed from R4; footprint (none) -> Resistor_SMD:R_0402_1005Metric
- R7: renamed from R3; footprint (none) -> Resistor_SMD:R_0402_1005Metric
- R8: renamed from R6; footprint (none) -> Resistor_SMD:R_0402_1005Metric
- R9: renamed from R2; footprint (none) -> Resistor_SMD:R_0402_1005Metric
- SW1, SW2: footprint (none) -> Button_Switch_SMD:SW_Tactile_SPST_NO_Straight_CK_PTS636Sx25SMTRLFS
- renumbered FLASH_MEMORY_8MB to FLASH_MEMORY_8MB1, RP2350B to RP2350B1
Connections:
- net +3V3: now also J2.1 (Pin_1)
- net GND: now also J4.A1 (GND), J4.A12 (GND), J4.B1 (GND), J4.B12 (GND), R1.2, R2.2
- net GPIO0: now also J2.2 (Pin_2)
- net GPIO1: now also J2.3 (Pin_3)
- net GPIO10: now also J2.12 (Pin_12)
- net GPIO11: now also J2.13 (Pin_13)
- net GPIO12: now also J2.14 (Pin_14)
- net GPIO13: now also J2.15 (Pin_15)
- net GPIO14: now also J2.16 (Pin_16)
- net GPIO15: now also J2.17 (Pin_17)
- net GPIO16: now also J2.18 (Pin_18)
- net GPIO17: now also J2.19 (Pin_19)
- net GPIO18: now also J2.20 (Pin_20)
- net GPIO19: now also J2.21 (Pin_21)
- net GPIO2: now also J2.4 (Pin_4)
- net GPIO20: now also J2.22 (Pin_22)
- net GPIO21: now also J2.23 (Pin_23)
- net GPIO22: now also J2.24 (Pin_24)
- net GPIO23: now also J2.25 (Pin_25)
- net GPIO24: now also J2.26 (Pin_26)
- net GPIO25: now also J3.26 (Pin_26)
- net GPIO26: now also J3.25 (Pin_25)
- net GPIO27: now also J3.24 (Pin_24)
- net GPIO28: now also J3.20 (Pin_20)
- net GPIO29: now also J3.19 (Pin_19)
- net GPIO3: now also J2.5 (Pin_5)
- net GPIO30: now also J3.18 (Pin_18)
- net GPIO31: now also J3.17 (Pin_17)
- net GPIO32: now also J3.16 (Pin_16)
- net GPIO33: now also J3.15 (Pin_15)
- net GPIO34: now also J3.14 (Pin_14)
- net GPIO35: now also J3.13 (Pin_13)
- net GPIO36: now also J3.12 (Pin_12)
- net GPIO37: now also J3.11 (Pin_11)
- net GPIO38: now also J3.10 (Pin_10)
- net GPIO39: now also J3.9 (Pin_9)
- net GPIO4: now also J2.6 (Pin_6)
- net GPIO40_ADC0: now also J3.8 (Pin_8)
- net GPIO41_ADC1: now also J3.7 (Pin_7)
- net GPIO42_ADC2: now also J3.6 (Pin_6)
- net GPIO43_ADC3: now also J3.5 (Pin_5)
- net GPIO44_ADC4: now also J3.4 (Pin_4)
- net GPIO45_ADC5: now also J3.3 (Pin_3)
- net GPIO46_ADC6: now also J3.2 (Pin_2)
- net GPIO47_ADC7: now also J3.1 (Pin_1)
- net GPIO5: now also J2.7 (Pin_7)
- net GPIO6: now also J2.8 (Pin_8)
- net GPIO7: now also J2.9 (Pin_9)
- net GPIO8: now also J2.10 (Pin_10)
- net GPIO9: now also J2.11 (Pin_11)
- net RUN: now also J3.21 (Pin_21)
- net SWCLK: now also J3.23 (Pin_23)
- net SWD: now also J3.22 (Pin_22)
- net USB_D+: now also J4.A6 (D+), J4.B6 (D+)
- net USB_D-: now also J4.A7 (D-), J4.B7 (D-)
- net VBUS: now also D1.1 (K)
- new net: D1.2 (A), J4.A4 (VBUS), J4.A9 (VBUS), J4.B4 (VBUS), J4.B9 (VBUS)
- new net: J4.A5 (CC1), R1.1
- new net: J4.B5 (CC2), R2.1
- no-connect marks 1 -> 3
Other:
- note added: "GPIO PINHEADER"
- note added: "MCU"
- note removed: "IOs"
- moved on the sheet: C1, C10, C11, C12, C13, C14, C15, C16, C17, C18, C19, C2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

Commit message: Update mcu.kicad_sch
Parts:
- removed R10, R11: 27, Resistor_SMD:R_0402_1005Metric, symbol Device:R
- removed R3, R5: DNF, Resistor_SMD:R_0402_1005Metric, symbol Device:R
- removed R4: 0, Resistor_SMD:R_0402_1005Metric, symbol Device:R
- removed R6, R8, R9: 1k, Resistor_SMD:R_0402_1005Metric, symbol Device:R
- removed R7: R3, Resistor_SMD:R_0402_1005Metric, symbol Device:R
- added R10, R11: 27, symbol Device:R_Small_US
- added R3: 33, symbol Device:R_Small_US
- added R3, R5: DNF, symbol Device:R_Small_US
- added R4: 0, symbol Device:R_Small_US
- added R6, R8, R9: 1k, symbol Device:R_Small_US
- D1: MPN NCP1117ST50T3G -> SM5817PL-TP
- J4: MPN (none) -> UJ20-C-H-G-SMT-1-P16-TR
- SW1, SW2: MPN (none) -> PTS636 SK43 SMTR LFS
- renumbered FLASH_MEMORY_8MB1 to FLASH_MEMORY_8MB
Connections:
- net +3.3V: now also R3.1
- net +3V3: now also R5.1
- net GND: now also J2.4 (Pin_4), R6.1
- net GPIO0: now also R3.1; no longer J2.2 (Pin_2)
- net GPIO1: no longer J2.3 (Pin_3)
- net GPIO2: now also RP2350B1.79 (GPIO2); no longer J2.4 (Pin_4)
- net GPIO25: no longer J3.26 (Pin_26)
- net GPIO26: no longer J3.25 (Pin_25)
- net GPIO27: now also J3.26 (Pin_26)
- net GPIO28: now also J3.25 (Pin_25)
- net GPIO4: no longer RP2350B1.79 (GPIO2)
- net QSPI_SS: now also R4.1
- net RUN: no longer RP2350B1.35 (RUN), SW2.2
- net USB_D+: now also R10.2
- net USB_D-: now also R11.2
- net VBUS: now also J2.3 (Pin_3)
- net XOUT: now also R9.2
- net at C10.1, RP2350B1.61 (VREG_AVDD): now also R3.2
- net at RP2350B1.66 (USB_DM): now also R11.1
- net at RP2350B1.67 (USB_DP): now also R10.1
- net at RP2350B1.75 (QSPI_SS): now also R8.2
- net at C5.2, Y1.3: now also R9.1
- net at SW2.1: now also R6.2
- net FLASH_SS: no longer names the net of FLASH_MEMORY_8MB.1 (/CS)
- net FLASH_SS: now also R3.2, R4.2, R5.2
- net USB_BOOT: no longer names the net of SW1.2
- net USB_BOOT: now also R8.1
- net VREG_LX: no longer names the net of L1.2, RP2350B1.63 (VREG_LX)
- new net: RP2350B1.35 (RUN), SW2.2
- new net +1V8: J2.2 (Pin_2)
Other:
- moved on the sheet: C4, C5, Y1

Commit message: Update mcu.kicad_sch
Parts:
- removed J2, J3: Conn_01x26_Pin, Connector_PinHeader_2.54mm:PinHeader_1x26_P2.54mm_Vertical, symbol Connector:Conn_01x26_Pin
- added J2: Conn_02x20_Counter_Clockwise, Connector_IDC:IDC-Header_2x20_P2.54mm_Vertical, symbol Connector_Generic:Conn_02x20_Counter_Clockwise
- RP2350B1: footprint (none) -> Footprints:RP2350B_QFN-80_EP_10.573x10.573_Pitch0.4mm
Connections:
- net +1V8: now also J2.2 (Pin_2)
- net +3V3: now also J2.1 (Pin_1)
- net GND: now also J2.21 (Pin_21)
- net GPIO1: now also J2.4 (Pin_4)
- net GPIO10: now also J2.13 (Pin_13)
- net GPIO11: now also J2.14 (Pin_14)
- net GPIO12: now also J2.15 (Pin_15)
- net GPIO13: now also J2.16 (Pin_16)
- net GPIO14: now also J2.17 (Pin_17)
- net GPIO15: now also J2.18 (Pin_18)
- net GPIO16: now also J2.19 (Pin_19)
- net GPIO17: now also J2.20 (Pin_20)
- net GPIO18: now also J2.40 (Pin_40)
- net GPIO19: now also J2.39 (Pin_39)
- net GPIO2: now also J2.5 (Pin_5)
- net GPIO20: now also J2.38 (Pin_38)
- net GPIO21: now also J2.37 (Pin_37)
- net GPIO22: now also J2.36 (Pin_36)
- net GPIO23: now also J2.35 (Pin_35)
- net GPIO24: now also J2.34 (Pin_34)
- net GPIO25: now also J2.33 (Pin_33)
- net GPIO26: now also J2.32 (Pin_32)
- net GPIO27: now also J2.31 (Pin_31)
- net GPIO28: now also J2.30 (Pin_30)
- net GPIO29: now also J2.29 (Pin_29)
- net GPIO3: now also J2.6 (Pin_6)
- net GPIO30: now also J2.28 (Pin_28)
- net GPIO31: now also J2.27 (Pin_27)
- net GPIO32: now also J2.26 (Pin_26)
- net GPIO33: now also J2.25 (Pin_25)
- net GPIO4: now also J2.7 (Pin_7)
- net GPIO5: now also J2.8 (Pin_8)
- net GPIO6: now also J2.9 (Pin_9)
- net GPIO7: now also J2.10 (Pin_10)
- net GPIO8: now also J2.11 (Pin_11)
- net GPIO9: now also J2.12 (Pin_12)
- net RUN: now also J2.24 (Pin_24)
- net SWCLK: now also J2.22 (Pin_22)
- net SWD: now also J2.23 (Pin_23)
- net VBUS: now also J2.3 (Pin_3)
Other:
- moved on the sheet: C4, C5, R9, Y1
