File: eco_devkit/debug_probe.kicad_sch (KiCad schematic)
At the start: 30 parts, among them J10 SWD Interface, J9 USB_C_Receptacle_USB2.0_16P, Y2 ABM8-272-T3

Commit message: Notate schematic.
Parts:
- renumbered D7 to D8, R35 to R38, R36 to R39, R37 to R40, R38 to R41, R39 to R42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
