File: eco_devkit/i2c_spi.kicad_sch (KiCad schematic)
At the start: 24 parts, among them J11 DISPLAY FFC, J12 Micro_SD_Card_Det1, Q5 T2N7002AK,LM, Q6 SL2301S, U3 LTR-329ALS-01, U4 MC3419

Commit message: Atribui footprints.
Parts:
- Q5, Q6: footprint (none) -> Package_TO_SOT_SMD:SOT-23-3
- R45, R46, R49, R50: footprint (none) -> Resistor_SMD:R_0402_1005Metric
- U3: footprint (none) -> EcoDevkit:LTR-329ALS-01_LTO
Changed lines of the file:
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@@
 			)
 		)
-		(property "Footprint" ""
+		(property "Footprint" "Resistor_SMD:R_0402_1005Metric"
 			(at 147.32 102.87 0)
 			(effects
@@
 			)
 		)
-		(property "Footprint" ""
+		(property "Footprint" "EcoDevkit:LTR-329ALS-01_LTO"
 			(at 52.07 157.48 0)
 			(effects
@@
 			)
 		)
-		(property "Footprint" ""
+		(property "Footprint" "Package_TO_SOT_SMD:SOT-23-3"
 			(at 156.21 90.17 0)
 			(effects
@@
 			)
 		)
-		(property "Footprint" ""
+		(property "Footprint" "Resistor_SMD:R_0402_1005Metric"
 			(at 34.29 74.93 0)
 			(effects
@@
 			)
 		)
-		(property "Footprint" ""
+		(property "Footprint" "Package_TO_SOT_SMD:SOT-23-3"
 			(at 156.21 68.58 0)
 			(effects
@@
 			)
 		)
-		(property "Footprint" ""
+		(property "Footprint" "Resistor_SMD:R_0402_1005Metric"
 			(at 121.92 62.23 0)
 			(effects
@@
 			)
 		)
-		(property "Footprint" ""
+		(property "Footprint" "Resistor_SMD:R_0402_1005Metric"
 			(at 147.32 83.82 0)
 			(effects

Commit message: Corrige footprints.
Parts:
- J10: renamed from J11; footprint Connector_FFC-FPC:Amphenol_F32R-1A7x1-11016_1x16-1MP_P0.5mm_Horizontal -> Connector_FFC-FPC:Amphenol_F32R-1A7x1-11028_1x28-1MP_P0.5mm_Horizontal
- renumbered J12 to J11
Changed lines of the file:
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@@
 		(dnp no)
 		(fields_autoplaced yes)
-		(property "Reference" "J12"
+		(property "Reference" "J11"
 			(at 241.935 57.15 0)
 			(effects
@@
 			(project "eco_devkit"
 				(path "/308cd3d6-c3d9-49fe-9127-06fda61df52b/18936539-b78a-4a13-b6a3-f93843840718"
-					(reference "J12")
+					(reference "J11")
 					(unit 1)
 				)
@@
 		(on_board yes)
 		(dnp no)
-		(property "Reference" "J11"
+		(property "Reference" "J10"
 			(at 94.996 57.658 0)
 			(effects
@@
 			)
 		)
-		(property "Footprint" "Connector_FFC-FPC:Amphenol_F32R-1A7x1-11016_1x16-1MP_P0.5mm_Horizontal"
+		(property "Footprint" "Connector_FFC-FPC:Amphenol_F32R-1A7x1-11028_1x28-1MP_P0.5mm_Horizontal"
 			(at 95.25 80.01 0)
 			(effects
@@
 			(project ""
 				(path "/308cd3d6-c3d9-49fe-9127-06fda61df52b/18936539-b78a-4a13-b6a3-f93843840718"
-					(reference "J11")
-					(unit 1)
-				)
+					(reference "J10")
+					(unit 1)
+				)
