File: eco_devkit/i2c_spi.kicad_sch (KiCad schematic)
At the start: 24 parts, among them J11 Micro_SD_Card_Det1, J13 DISPLAY FFC, Q7 T2N7002AK,LM, Q8 SL2301S, U3 LTR-329ALS-01, U4 MC3419

Commit message: footprint completed
Parts:
- Q5: renamed from Q7; footprint Package_TO_SOT_SMD:SOT-23 -> Package_TO_SOT_SMD:SOT-23-3
- R46: renamed from R56; footprint (none) -> Resistor_SMD:R_0402_1005Metric
- R47: renamed from R54; footprint (none) -> Resistor_SMD:R_0402_1005Metric
- R48: renamed from R55; footprint (none) -> Resistor_SMD:R_0402_1005Metric
- R49: renamed from R53; footprint (none) -> Resistor_SMD:R_0402_1005Metric
- renumbered C50 to C41, C47 to C42, C53 to C43, C54 to C44, C57 to C45, C56 to C46, C55 to C47, C51 to C48, C52 to C49, J11 to J10, J13 to J11, Q8 to Q6, R51 to R42, R52 to R43, R47 to R44, R48 to R45, U3 to U2, U4 to U3
Connections:
- net +3V3: now also C41.2, J10.4 (VDD)
- net GND: now also J11.12 (BS2); no longer J11.1 (NC/GND)
- no-connect marks 7 -> 8
Other:
- moved on the sheet: Q5, U2

Commit message: Placement v1.
Parts:
- J11: footprint EcoDevkit:AMPHENOL_SFV28R-2STE1HLF -> EcoDevkit:FPC_30
Changed lines of the file:
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@@
 			)
 		)
-		(property "Footprint" "EcoDevkit:AMPHENOL_SFV28R-2STE1HLF"
+		(property "Footprint" "EcoDevkit:FPC_30"
 			(at 184.15 78.74 0)
 			(effects
