File: eco_devkit/analog_peripherals.kicad_sch (KiCad schematic)
At the start: 17 parts, among them J6 ADC_SEL1, J7 ADC_SEL1, J8 ADC_SEL1, U1 LM324

Commit message: Corrige footprints.
Parts:
- renumbered J6 to J5, J7 to J6, J8 to J7
Changed lines of the file:
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@@
 		(dnp no)
 		(fields_autoplaced yes)
-		(property "Reference" "J7"
+		(property "Reference" "J6"
 			(at 80.01 88.2649 90)
 			(effects
@@
 			(project "eco_devkit"
 				(path "/308cd3d6-c3d9-49fe-9127-06fda61df52b/a3f9a86b-c305-4ba8-be31-b3cd3a950ab4"
-					(reference "J7")
+					(reference "J6")
 					(unit 1)
 				)
@@
 		(dnp no)
 		(fields_autoplaced yes)
-		(property "Reference" "J6"
+		(property "Reference" "J5"
 			(at 45.72 88.2649 90)
 			(effects
@@
 			(project ""
 				(path "/308cd3d6-c3d9-49fe-9127-06fda61df52b/a3f9a86b-c305-4ba8-be31-b3cd3a950ab4"
-					(reference "J6")
+					(reference "J5")
 					(unit 1)
 				)
@@
 		(dnp no)
 		(fields_autoplaced yes)
-		(property "Reference" "J8"
+		(property "Reference" "J7"
 			(at 123.19 78.1049 90)
 			(effects
@@
 			(project "eco_devkit"
 				(path "/308cd3d6-c3d9-49fe-9127-06fda61df52b/a3f9a86b-c305-4ba8-be31-b3cd3a950ab4"
-					(reference "J8")
-					(unit 1)
-				)
+					(reference "J7")
+					(unit 1)
+				)

Commit message: footprint completed
Parts:
- removed R35: 0, Resistor_SMD:R_0402_1005Metric, symbol Device:R_Small_US
- removed R36: 1M, Resistor_SMD:R_0402_1005Metric, symbol Device:R_Small_US
- removed R37: 1k, Resistor_SMD:R_0402_1005Metric, symbol Device:R_Small_US
- removed RV3: 100K, EcoDevkit:TRIM_TC33X-2-203E, symbol Device:R_Potentiometer_Trim_US
- removed U1: LM324, Package_SO:TSSOP-14_4.4x5mm_P0.65mm, symbol Amplifier_Operational:LM324
Connections:
- net MIC_AMP is gone; now on net MIC_OUT: C25.2
- no-connect marks 1 -> 0
Other:
- note removed: "AMPLIFIER CIRCUIT (DNF)"
- moved on the sheet: C25, J5, J6, J7, MK1, R30, R31, R32, R33, R34, RV1, RV2
