File: eco_devkit/analog_peripherals.kicad_sch (KiCad schematic)
At the start: 0 parts

Commit message: Update layout
Parts:
- added C25: 1u, Capacitor_SMD:C_0402_1005Metric, symbol Device:C
- added J5, J6, J7: ADC_SEL1, Connector_PinSocket_2.54mm:PinSocket_1x02_P2.54mm_Vertical, symbol Connector:Conn_01x02_Pin
- added MK1: MIC, EcoDevkit:MIC_CMEJ-0415-42-P, symbol EcoDevkit:Microphone_Condenser
- added R30, R31: 1k, Resistor_SMD:R_0402_1005Metric, symbol Device:R_Small_US
- added R32: 33k, Resistor_SMD:R_0402_1005Metric, symbol Device:R_Small_US
- added R33: 500k, OptoDevice:R_LDR_5.1x4.3mm_P3.4mm_Vertical, symbol Sensor_Optical:LDR07
- added R34: 2.2k, Resistor_SMD:R_0402_1005Metric, symbol Device:R_Small_US
- added RV1, RV2: 100k, EcoDevkit:TRIM_TC33X-2-203E, symbol Device:R_Potentiometer_Trim_US
Connections:
- new net: R30.2, RV1.1
- new net: J5.2 (Pin_2), RV1.2
- new net: J6.2 (Pin_2), RV2.2
- new net: R31.2, RV2.1
- new net: J7.2 (Pin_2), R32.2, R33.1
- new net: C25.1, MK1.1 (+), R34.2
- new net +3V3: R30.1, R31.1, R32.1, R34.1
- new net GND: MK1.2 (-), R33.2, RV1.3, RV2.3
- new net LDR_IN: J7.1 (Pin_1)
- new net MIC_OUT: C25.2
- new net TRIM1_IN: J6.1 (Pin_1)
- new net TRIM2_IN: J5.1 (Pin_1)
Other:
- note added: "ANALOG PERIPHERALS"
- note added: "GENERIC ANALOG"
- note added: "MICROPHONE ELECTRET"

Commit message: Placement v1.
Parts:
- J5, J6, J7: footprint Connector_PinSocket_2.54mm:PinSocket_1x02_P2.54mm_Vertical -> Connector_PinHeader_2.54mm:PinHeader_1x02_P2.54mm_Vertical
Changed lines of the file:
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@@
 			)
 		)
-		(property "Footprint" "Connector_PinSocket_2.54mm:PinSocket_1x02_P2.54mm_Vertical"
+		(property "Footprint" "Connector_PinHeader_2.54mm:PinHeader_1x02_P2.54mm_Vertical"
 			(at 116.84 92.71 0)
 			(effects
@@
 			)
 		)
-		(property "Footprint" "Connector_PinSocket_2.54mm:PinSocket_1x02_P2.54mm_Vertical"
+		(property "Footprint" "Connector_PinHeader_2.54mm:PinHeader_1x02_P2.54mm_Vertical"
 			(at 82.55 92.71 0)
 			(effects
@@
 			)
 		)
-		(property "Footprint" "Connector_PinSocket_2.54mm:PinSocket_1x02_P2.54mm_Vertical"
+		(property "Footprint" "Connector_PinHeader_2.54mm:PinHeader_1x02_P2.54mm_Vertical"
 			(at 160.02 82.55 0)
 			(effects

Commit message: Finaliza projeto
Parts:
- added J12: ADC_SEL1, Connector_PinHeader_2.54mm:PinHeader_1x02_P2.54mm_Vertical, symbol Connector:Conn_01x02_Pin
Connections:
- net MIC_OUT: now also J12.1 (Pin_1); no longer C25.2
- new net: C25.2, J12.2 (Pin_2)
Changed lines of the file:
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@@
+	(wire
+		(pts
+			(xy 205.74 88.9) (xy 214.63 88.9)
+		)
+		(stroke
+			(width 0)
+			(type default)
+		)
+	)
 	(wire
 		(pts
@@
 	(wire
 		(pts
-			(xy 205.74 88.9) (xy 227.33 88.9)
+			(xy 157.48 87.63) (xy 157.48 88.9)
 		)
 		(stroke
@@
 	(wire
 		(pts
-			(xy 157.48 87.63) (xy 157.48 88.9)
+			(xy 146.05 85.09) (xy 146.05 88.9)
 		)
 		(stroke
@@
 	(wire
 		(pts
-			(xy 146.05 85.09) (xy 146.05 88.9)
+			(xy 160.02 87.63) (xy 160.02 88.9)
 		)
 		(stroke
@@
 	(wire
 		(pts
-			(xy 160.02 87.63) (xy 160.02 88.9)
+			(xy 104.14 87.63) (xy 104.14 95.25)
 		)
 		(stroke
@@
 	(wire
 		(pts
-			(xy 104.14 87.63) (xy 104.14 95.25)
+			(xy 116.84 97.79) (xy 116.84 99.06)
 		)
 		(stroke
@@
 	(wire
 		(pts
-			(xy 116.84 97.79) (xy 116.84 99.06)
+			(xy 69.85 87.63) (xy 69.85 95.25)
 		)
 		(stroke
@@
 	(wire
 		(pts
-			(xy 69.85 87.63) (xy 69.85 95.25)
+			(xy 217.17 88.9) (xy 227.33 88.9)
 		)
 		(stroke
@@
 					(unit 1)
 				)
+			)
+		)
+	)
+	(symbol
+		(lib_id "Connector:Conn_01x02_Pin")
+		(at 217.17 83.82 270)
+		(unit 1)
+		(exclude_from_sim no)
+		(in_bom yes)
+		(on_board yes)
+		(dnp no)
+		(fields_autoplaced yes)
+		(property "Reference" "J12"
+			(at 218.44 83.1849 90)
+			(effects
+				(font
+					(size 1.27 1.27)
+				)
+				(justify left)
+			)
+		)
+		(property "Value" "ADC_SEL1"
+			(at 218.44 85.7249 90)
+			(effects
+				(font
+					(size 1.27 1.27)
+				)
+				(justify left)
+			)
+		)
+		(property "Footprint" "Connector_PinHeader_2.54mm:PinHeader_1x02_P2.54mm_Vertical"
+			(at 217.17 83.82 0)
+			(effects
+				(font
+					(size 1.27 1.27)
+				)
+				(hide yes)
+			)
+		)
+		(property "Datasheet" "~"
+			(at 217.17 83.82 0)
+			(effects
+				(font
+					(size 1.27 1.27)
+				)
+				(hide yes)
+			)
+		)
+		(property "Description" "Generic connector, single row, 01x02, script generated"
+			(at 217.17 83.82 0)
+			(effects
+				(font
+					(size 1.27 1.27)
+				)
+				(hide yes)
+			)
+		)
+		(pin "2"
+		)
+		(pin "1"
+		)
+		(instances
+			(project "eco_devkit"
+				(path "/308cd3d6-c3d9-49fe-9127-06fda61df52b/a3f9a86b-c305-4ba8-be31-b3cd3a950ab4"
+					(reference "J12")
+					(unit 1)
+				)
