File: eco_devkit/eco_devkit.kicad_pcb (KiCad board)
At the start: 2 copper layers, 41 parts, among them J1 USB_C_Receptacle_USB2.0_16P, J2 Conn_02x20_Counter_Clockwise, SW1 BOOT, SW2 RESET, Y1 Crystal_GND24

Commit message: feat: placement of MCU passive components and crystal
Parts:
- moved C20 195.2 mm to (269.5, 72.0), turned to -90 degrees
- moved FLASH_MEMORY_8MB1 192.8 mm to (261.1, 46.9)
- moved C19 191.7 mm to (266.0, 71.9), turned to -90 degrees
- moved J1 189.3 mm to (189.8, 150.3)
- moved C18 188.2 mm to (262.5, 71.9), turned to -90 degrees
- moved C17 184.7 mm to (259.0, 72.0), turned to -90 degrees
- moved C16 181.3 mm to (255.5, 72.0), turned to -90 degrees
- moved C15 180.5 mm to (252.0, 72.0), turned to -90 degrees
- moved C10 179.1 mm to (247.5, 64.5), turned to 90 degrees
- moved C8 178.7 mm to (247.0, 79.5), turned to -90 degrees
- moved C14 177.0 mm to (248.5, 72.0), turned to -90 degrees
- moved C6 176.4 mm to (245.0, 60.5), turned to 90 degrees
- moved C9 176.1 mm to (244.5, 79.5), turned to -90 degrees
- moved C13 173.5 mm to (245.0, 72.0), turned to -90 degrees
- moved C7 171.5 mm to (240.0, 63.0)
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Connections:
- RP2350B1 pad 30: /MCU/XOUT -> /MCU/XIN

Commit message: feat: MCU placement and routing of power and signal connections
Parts:
- moved J2 205.5 mm to (228.5, 28.7)
- moved J1 139.8 mm to (256.0, 27.2), turned to 180 degrees
- moved NCP1 139.2 mm to (246.1, 31.1)
- moved R3 107.8 mm to (257.7, 36.3)
- moved R4 106.7 mm to (253.7, 36.3), turned to 180 degrees
- moved R2 92.2 mm to (244.3, 41.8)
- moved R1 90.1 mm to (244.3, 42.9)
- moved R5 89.5 mm to (244.3, 40.8)
- moved D1 88.8 mm to (244.7, 37.4)
- moved C4 68.0 mm to (254.3, 41.4)
- moved C3 54.7 mm to (241.2, 35.1), turned to 90 degrees
- moved C5 54.7 mm to (241.0, 30.7), turned to 90 degrees
- moved C1 40.8 mm to (253.6, 70.0), turned to 90 degrees
- moved C2 38.4 mm to (248.2, 69.9), turned to -90 degrees
- moved R6 37.9 mm to (254.8, 70.0), turned to 90 degrees
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Connections:
- J2 pad 10: /MCU/GPIO6 -> PIN_LIGHT_SENS_SDA
- J2 pad 11: PIN_WIFI_RESET_BL -> SWD
- J2 pad 12: PIN_WIFI_RX -> PIN_LIGHT_SENS_SCL
- J2 pad 13: PIN_WIFI_TX -> /MCU/GPIO24
- J2 pad 14: DISPLAY_SCK -> /MCU/GPIO6
- J2 pad 15: DISPLAY_MOSI -> GPIO41_ADC1
- J2 pad 16: DISPLAY_RST -> PIN_WIFI_RESET_BL
- J2 pad 17: DISPLAY_EN -> GPIO43_ADC3
- J2 pad 18: /MCU/GPIO14 -> PIN_WIFI_RX
- J2 pad 19: /MCU/GPIO15 -> PIN_BUZZER
- J2 pad 20: /MCU/GPIO16 -> PIN_WIFI_TX
- J2 pad 22: SWD -> DISPLAY_SCK
- J2 pad 24: GPIO43_ADC3 -> DISPLAY_MOSI
- J2 pad 26: GPIO45_ADC5 -> DISPLAY_RST
- J2 pad 28: GPIO43_ADC3 -> DISPLAY_EN
- J2 pad 30: GPIO41_ADC1 -> /MCU/GPIO14
- J2 pad 32: PIN_BUZZER -> /MCU/GPIO15
- J2 pad 34: /MCU/GPIO24 -> /MCU/GPIO16
- J2 pad 36: GPIO21 -> /MCU/GPIO17
- J2 pad 37: ACCEL_MISO -> GPIO21
- J2 pad 4: GND -> POBRE_GPIO5/UART_RX
- J2 pad 40: /MCU/GPIO17 -> ACCEL_MISO
- J2 pad 5: POBRE_GPIO5/UART_RX -> GND
- J2 pad 7: /MCU/GPIO3 -> GPIO45_ADC5
- J2 pad 8: PIN_LIGHT_SENS_SDA -> /MCU/GPIO3
- J2 pad 9: PIN_LIGHT_SENS_SCL -> GPIO43_ADC3
Routing:
- net +3V3: track 0.00 -> 44.0 mm
- net POBRE_GPIO5/UART_RX: track 0.00 -> 30.6 mm
- net /MCU/GPIO2: track 0.00 -> 29.0 mm
- net ACCEL_SCK: track 0.00 -> 28.8 mm
- net /MCU/GPIO3: track 0.00 -> 27.2 mm
- net ACCEL_MISO: track 0.00 -> 26.3 mm
- net PIN_LIGHT_SENS_SDA: track 0.00 -> 25.5 mm
- net ACCEL_MOSI: track 0.00 -> 24.4 mm
- net PIN_LIGHT_SENS_SCL: track 0.00 -> 24.1 mm
- net /MCU/GPIO17: track 0.00 -> 23.4 mm
- net /MCU/GPIO16: track 0.00 -> 22.5 mm
- net /MCU/GPIO15: track 0.00 -> 21.8 mm
- net /MCU/GPIO6: track 0.00 -> 21.8 mm
- net /MCU/GPIO14: track 0.00 -> 20.9 mm
- net DISPLAY_EN: track 0.00 -> 20.0 mm
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- added copper zone on F.Cu, net (none)
- added copper zone on F.Cu, net +3V3
